File: pcb/EAGLE/Thor_v1.sch (EAGLE design)
At the start: 213 parts, among them P0.1 39-30-02, P0.2 39-30-02, P1 39-30-02, P1.1 39-30-02, P1.2 39-30-02, P10 39-30-02, P11 39-30-02, P12 39-30-02, P13 39-30-02, P14 39-30-02, P15 39-30-02, P16 39-30-02, P17 39-30-02, P19 39-30-02, P2.1 39-30-02, P2.2 39-30-02, P20 39-30-02, P21 39-30-02, P22 39-30-02, P23 39-30-02, P24 39-30-02, P25 39-30-02, P26 39-30-02, P27 39-30-02, P28 39-30-02, P29 39-30-02, P3 39-30-02, P30 39-30-02, P31 39-30-02, P32 39-30-02, P33 39-30-02, P34 39-30-02, P37 39-30-02, P38 39-30-02, P39 39-30-02, P4 39-30-02, P40 39-30-02, P41 39-30-02, P42 39-30-02, P43 39-30-02, P44 39-30-02, P45 39-30-02, P46 39-30-02, P47 39-30-02, P48 39-30-02, P49 39-30-02, P5 39-30-02, P50 39-30-02, P51 39-30-02, P52 39-30-02, P6 39-30-02, P7 39-30-02, P8 39-30-02, P9 39-30-02, Q1 T460, Q10 T460, Q11 T460, Q12 T460, Q13 T460, Q14 T460, Q15 T460, Q16 T460, Q17 T460, Q18 T460, Q19 T460, Q2 T460, Q20 T460, Q21 T460, Q22 T460, Q23 T460, Q24 T460, Q25 T460, Q26 T460, Q27 T460, Q28 T460, Q29 T460, Q3 T460, Q30 T460, Q31 T460, Q32 T460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

Commit message: more work on initial design
Connections:
- net 22: now also U2.22
- net 23: now also U2.23
- net 24: now also U2.24
- net 26: now also U2.26
- net 27: now also U2.27
- net 28: now also U2.28
- net 29: now also U2.29
- net 30: now also U2.30
- net 31: now also U2.31
- net 32: now also U2.32
- net 33: now also U2.33
- net 34: now also U2.34
- net 35: now also U2.35
- net 36: now also U2.36
- net 37: now also U2.37
- net 38: now also U2.38
- net 39: now also U2.39
- net N$9: now also U2.25
Other:
- note removed: "2x I2C busses"
- note removed: "Power Rail on Single Side"
- moved on the sheet: I2C-1, I2C-2, I2C-3, P-P1, P-P2, P0.1, P0.2, P1-P2, P1.1, P1.2, P2.1, P2.2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
